Commit message: детекция объекта / захват объекта

File: ros_ws/src/smart_arm_demo/urdf/ur5_with_gripper.xacro (robot description, xacro)
@@ -1,4 +1,4 @@
 <?xml version="1.0"?>
-<robot xmlns:xacro="http://www.ros.org/wiki/xacro" name="ur5_with_gripper">
+<robot xmlns:xacro="http://www.ros.org/wiki/xacro" name="ur5">
   <xacro:include filename="$(find ur_description)/urdf/inc/ur5_macro.xacro"/>
   <material name="mat_black">
@@ -35,10 +35,4 @@
       <material name="mat_black"/>
     </visual>
-    <collision>
-      <origin xyz="0 0 0.03" rpy="0 0 0"/>
-      <geometry>
-        <box size="0.10 0.16 0.02"/>
-      </geometry>
-    </collision>
   </link>
   <joint name="gripper_base_joint" type="fixed">
@@ -64,10 +58,4 @@
       <material name="mat_green"/>
     </visual>
-    <collision>
-      <origin xyz="0 0 0.02" rpy="0 0 0"/>
-      <geometry>
-        <box size="0.02 0.01 0.10"/>
-      </geometry>
-    </collision>
   </link>
   <link name="finger_right_link">
@@ -84,15 +72,9 @@
       <material name="mat_green"/>
     </visual>
-    <collision>
-      <origin xyz="0 0 0.02" rpy="0 0 0"/>
-      <geometry>
-        <box size="0.02 0.01 0.10"/>
-      </geometry>
-    </collision>
   </link>
   <joint name="finger_left_joint" type="prismatic">
-    <parent link="wrist_3_link"/>
+    <parent link="gripper_base_link"/>
     <child link="finger_left_link"/>
-    <origin xyz="0.12 0.06 0" rpy="0 0 0"/>
+    <origin xyz="0.0 0.06 0" rpy="0 0 0"/>
     <axis xyz="0 -1 0"/>
     <limit lower="0.0" upper="0.055" effort="60" velocity="0.25"/>
@@ -100,7 +82,7 @@
   </joint>
   <joint name="finger_right_joint" type="prismatic">
-    <parent link="wrist_3_link"/>
+    <parent link="gripper_base_link"/>
     <child link="finger_right_link"/>
-    <origin xyz="0.12 -0.06 0" rpy="0 0 0"/>
+    <origin xyz="0.0 -0.06 0" rpy="0 0 0"/>
     <axis xyz="0 1 0"/>
     <limit lower="0.0" upper="0.055" effort="60" velocity="0.25"/>

Commit message: fix логики движения за объектом

File: ros_ws/src/smart_arm_demo/urdf/ur5_with_gripper.xacro (robot description, xacro)
@@ -1,4 +1,4 @@
 <?xml version="1.0"?>
-<robot xmlns:xacro="http://www.ros.org/wiki/xacro" name="ur5">
+<robot xmlns:xacro="http://www.ros.org/wiki/xacro" name="ur5_robot">
   <xacro:include filename="$(find ur_description)/urdf/inc/ur5_macro.xacro"/>
   <material name="mat_black">
@@ -35,9 +35,12 @@
       <material name="mat_black"/>
     </visual>
+    <!-- No URDF collision on palm: a palm box makes MoveIt report START_STATE_IN_COLLISION at home. -->
+    <!-- Gazebo contact still uses finger collision + attach node. -->
   </link>
+  <!-- Без смещения 0.12 м: основание захвата совпадает с фланцем последней оси (wrist_3). При наличии tool0 в вашей сборке можно сменить parent на tool0. -->
   <joint name="gripper_base_joint" type="fixed">
     <parent link="wrist_3_link"/>
     <child link="gripper_base_link"/>
-    <origin xyz="0.12 0 0.00" rpy="0 0 0"/>
+    <origin xyz="0 0 0" rpy="0 0 0"/>
   </joint>
   <gazebo reference="gripper_base_joint">
@@ -58,4 +61,10 @@
       <material name="mat_green"/>
     </visual>
+    <collision>
+      <origin xyz="0 0 0.02" rpy="0 0 0"/>
+      <geometry>
+        <box size="0.014 0.006 0.075"/>
+      </geometry>
+    </collision>
   </link>
   <link name="finger_right_link">
@@ -72,4 +81,10 @@
       <material name="mat_green"/>
     </visual>
+    <collision>
+      <origin xyz="0 0 0.02" rpy="0 0 0"/>
+      <geometry>
+        <box size="0.014 0.006 0.075"/>
+      </geometry>
+    </collision>
   </link>
   <joint name="finger_left_joint" type="prismatic">
@@ -110,15 +125,22 @@
   </transmission>
   <gazebo reference="finger_left_link">
-    <mu1>50</mu1>
-    <mu2>50</mu2>
-    <kp>100000</kp>
-    <kd>5</kd>
+    <mu1>80</mu1>
+    <mu2>80</mu2>
+    <kp>1000000</kp>
+    <kd>100</kd>
     <selfCollide>false</selfCollide>
   </gazebo>
   <gazebo reference="finger_right_link">
-    <mu1>50</mu1>
-    <mu2>50</mu2>
-    <kp>100000</kp>
-    <kd>5</kd>
+    <mu1>80</mu1>
+    <mu2>80</mu2>
+    <kp>1000000</kp>
+    <kd>100</kd>
+    <selfCollide>false</selfCollide>
+  </gazebo>
+  <gazebo reference="gripper_base_link">
+    <mu1>80</mu1>
+    <mu2>80</mu2>
+    <kp>1000000</kp>
+    <kd>100</kd>
     <selfCollide>false</selfCollide>
   </gazebo>
